File: schematic/boost_converter.kicad_sch (KiCad schematic)
At the start: 10 parts, among them Q1 NMOS, Q2 PN2222A

Commit message: Add buck converter to schematic
Changed lines of the file:
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@@
     (stroke (width 0) (type default))
+  )
+  (text_box "Ideally, this should be a pullup network instead of a pulldown since the NMOS transistor being on for long periods of time could damage the transistor since it presents as a short to ground."
+    (at 19.05 86.36 0) (size 40.64 15.24)
+    (stroke (width 0) (type default))
+    (fill (type none))
+    (effects (font (size 1.27 1.27)) (justify left top))
   )
   (hierarchical_label "V_{fdbk}" (shape input) (at 133.35 71.12 0) (fields_autoplaced)
